Commit message: add camera sim,but not succeed

File: rm_description/urdf/hero/hero.urdf.xacro (robot description, xacro)
@@ -8,4 +8,5 @@
   <xacro:arg name="roller_type" default="realistic"/>
   <xacro:arg name="load_laser" default="false"/>
+  <xacro:arg name="load_camera" default="false"/>
   <xacro:if value="$(arg load_chassis)">
     <xacro:include filename="$(find rm_description)/urdf/hero/chassis.urdf.xacro"/>
@@ -33,8 +34,11 @@
     </xacro:unless>
   </xacro:if>
+  <xacro:include filename="$(find rm_description)/urdf/sensor/head.urdf.xacro" />
+  <xacro:include filename="$(find rm_description)/urdf/sensor/sensor.urdf.xacro" />
   <xacro:if value="$(arg load_laser)">
-    <xacro:include filename="$(find rm_description)/urdf/sensor/head.urdf.xacro" />
-    <xacro:include filename="$(find rm_description)/urdf/sensor/laser.urdf.xacro" />
     <xacro:include filename="$(find rm_description)/urdf/sensor/laser_sim.urdf.xacro" />
   </xacro:if>
+  <xacro:if value="$(arg load_camera)">
+    <xacro:include filename="$(find rm_description)/urdf/sensor/camera_sim.urdf.xacro" />
+  </xacro:if>
 </robot>

File: rm_description/urdf/sensor/laser_sim.urdf.xacro (robot description, xacro)
@@ -1,6 +1,5 @@
 <robot name="my_sensors" xmlns:xacro="http://wiki.ros.org/xacro">
   <!-- 雷达 -->
-  <gazebo reference="laser">
-    <!-- 这里，把雷达映射到了laser这个link上 -->
+  <gazebo reference="sensor">
     <sensor type="ray" name="rplidar">
       <pose>0 0 0 0 0 0</pose>
@@ -29,5 +28,5 @@
       <plugin name="gazebo_rplidar" filename="libgazebo_ros_laser.so">
         <topicName>/scan</topicName>
-        <frameName>laser</frameName>
+        <frameName>sensor</frameName>
       </plugin>
     </sensor>

File: rm_description/urdf/sensor/sensor.urdf.xacro (robot description, xacro)
@@ -1,3 +1,3 @@
-<robot name="laser" xmlns:xacro="http://wiki.ros.org/xacro">
+<robot name="sensor" xmlns:xacro="http://wiki.ros.org/xacro">
     <!-- 雷达支架 -->
     <xacro:property name="support_length" value="0.15" /> <!-- 支架长度 -->
@@ -41,5 +41,5 @@
     <xacro:property name="laser_m" value="0.1" /> <!-- 雷达质量 -->
     <!-- 雷达关节以及link -->
-    <link name="laser">
+    <link name="sensor">
         <visual>
             <geometry>
@@ -59,8 +59,8 @@
     <joint name="laser2support" type="fixed">
         <parent link="support" />
-        <child link="laser" />
+        <child link="sensor" />
         <origin xyz="${laser_x} ${laser_y} ${laser_z}" />
     </joint>
-    <gazebo reference="laser">
+    <gazebo reference="sensor">
         <material>Gazebo/Black</material>
     </gazebo>

Commit message: realsense can use,planner not succeed

File: rm_description/urdf/hero/hero.urdf.xacro (robot description, xacro)
@@ -8,5 +8,6 @@
   <xacro:arg name="roller_type" default="realistic"/>
   <xacro:arg name="load_laser" default="false"/>
-  <xacro:arg name="load_camera" default="true"/>
+  <xacro:arg name="load_camera" default="false"/>
+  <xacro:arg name="realsense" default="true"/>
   <xacro:if value="$(arg load_chassis)">
     <xacro:include filename="$(find rm_description)/urdf/hero/chassis.urdf.xacro"/>
@@ -42,3 +43,10 @@
     <xacro:include filename="$(find rm_description)/urdf/sensor/camera_sim.urdf.xacro" />
   </xacro:if>
+  <xacro:if value="$(arg realsense)">
+    <xacro:include filename="$(find realsense_ros_gazebo)/xacro/tracker.xacro"/>
+    <xacro:include filename="$(find realsense_ros_gazebo)/xacro/depthcam.xacro"/>
+    <xacro:realsense_d435 sensor_name="d435" parent_link="base_link" rate="10">
+      <origin rpy="0 0 0 " xyz="0.18 0 0.3"/>
+    </xacro:realsense_d435>
+  </xacro:if>
 </robot>

Commit message: realsense + move_base ok

File: rm_description/urdf/hero/hero.urdf.xacro (robot description, xacro)
@@ -39,5 +39,5 @@
     <xacro:include filename="$(find realsense_ros_gazebo)/xacro/depthcam.xacro"/>
     <xacro:realsense_d435 sensor_name="d435" parent_link="base_link" rate="10">
-      <origin rpy="0 0 0 " xyz="0.18 0 0.3"/>
+      <origin rpy="0 0.26 0 " xyz="0.18 0 0.3"/>
     </xacro:realsense_d435>
   </xacro:if>
